Commit message: created wheels and robot base

File: src/simulation/robot_description/urdf/robot.xacro (robot description, xacro)
@@ -1,44 +1,46 @@
 <?xml version="1.0"?>
 <robot name="beagle_robot" xmlns:xacro="http://www.ros.org/wiki/xacro">
-	<xacro:property name="PI" value="3.1415926535897931"/>
-	<xacro:property name="chassisHeight" value="0.1"/>
-	<xacro:property name="chassisLength" value="0.4"/>
-	<xacro:property name="chassisWidth" value="0.2"/>
-	<xacro:property name="chassisMass" value="50"/>
-	<xacro:property name="casterRadius" value="0.05"/>
-	<xacro:property name="casterMass" value="5"/>
-	<xacro:property name="wheelWidth" value="0.05"/>
-	<xacro:property name="wheelRadius" value="0.1"/>
-	<xacro:property name="wheelPos" value="0.2"/>
-	<xacro:property name="wheelMass" value="5"/>
-	<xacro:property name="cameraSize" value="0.05"/>
-	<xacro:property name="cameraMass" value="0.1"/>
-	<xacro:include filename="$(find robot_description)/urdf/robot.gazebo" />
+	<property name="PI" value="3.1415926535897931"/>
+	<property name="robotWidth" value="0.28"/>
+	<property name="robotLength" value="0.27"/>
+	<property name="robotHeight" value="0.35"/>
+	<property name="wheelRadius" value="0.03"/>
+	<property name="wheelLength" value="0.01"/>
 	<xacro:include filename="$(find robot_description)/urdf/materials.xacro" />
-	<xacro:include filename="$(find robot_description)/urdf/macros.xacro" />
-	<link name="footprint" />
-	<joint name="base_joint" type="fixed">
-		<parent link="footprint"/>
-		<child link="chassis"/>
+	<link name="base_link">
+		<visual>
+			<geometry>
+				<box size="${robotWidth} ${robotLength} ${robotHeight}"/>
+			</geometry>
+			<material name="green"/>
+		</visual>
+	</link>
+	<link name="left_wheel">
+		<visual>
+			<geometry>
+				<cylinder radius="${wheelRadius}" length="${wheelLength}"/>
+			</geometry>
+			<material name="blue"/>
+		</visual>
+	</link>
+	<link name="right_wheel">
+		<visual>
+			<geometry>
+				<cylinder radius="${wheelRadius}" length="${wheelLength}"/>
+			</geometry>
+			<material name="red"/>
+		</visual>
+	</link>
+	<joint name="base_link_right_wheel" type="continuous">
+		<origin xyz="0.1 0.0 ${-robotHeight/2}" rpy="0.0 ${PI/2} 0.0"/>
+		<parent link="base_link"/>
+		<child link="right_wheel"/>
+		<axis xyz="0.0 0.0 1.0"/>
 	</joint>
-	<link name='chassis'>
-		<collision>
-			<origin xyz="0 0 ${wheelRadius}" rpy="0 0 0"/>
-			<geometry>
-				<box size="${chassisLength} ${chassisWidth} ${chassisHeight}"/>
-			</geometry>
-		</collision>
-		<visual>
-			<origin xyz="0 0 ${wheelRadius}" rpy="0 0 0"/>
-			<geometry>
-				<box size="${chassisLength} ${chassisWidth} ${chassisHeight}"/>
-			</geometry>
-			<material name="orange"/>
-		</visual>
-		<inertial>
-			<origin xyz="0 0 ${wheelRadius}" rpy="0 0 0"/>
-			<mass value="${chassisMass}"/>
-			<box_inertia m="${chassisMass}" x="${chassisLength}" y="${chassisWidth}" z="${chassisHeight}"/>
-		</inertial>
-	</link>
-</robot>>
+	<joint name="base_link_left_wheel" type="continuous">
+		<origin xyz="-0.1 0.0 ${-robotHeight/2}" rpy="0.0 ${PI/2} 0.0"/>
+		<parent link="base_link"/>
+		<child link="left_wheel"/>
+		<axis xyz="0.0 0.0 1.0"/>
+	</joint>
+</robot>
