Commit message: robot spawn fixed

File: src/simulation/beagle_description/urdf/beagle_robot.xacro (robot description, xacro)
@@ -22,4 +22,9 @@
 			</geometry>
 		</collision>
+		<inertial>
+			<mass value="1.0"/>
+			<!-- TODO -->
+			<inertia ixx="0.015" iyy="0.0375" izz="0.0375" ixy="0" ixz="0" iyz="0"/>
+		</inertial>
 	</link>
 	<link name="left_wheel">
